Commit message: TF coordinate frames; rviz

File: catkin_ws/src/desktopquad_sim/agents/chiny/chiny.xacro (robot description, xacro)
@@ -14,5 +14,5 @@
     <inertial>
       <mass value="${mass}" />  <!-- [kg] -->
-      <origin xyz="0 0 0" />
+      <origin xyz="0 0 0.005" />
       <xacro:insert_block name="body_inertia" />
     </inertial>
